File: Solenoid Board.brd (EAGLE design)
At the start: 76.2 x 31.8 mm, 38 parts, among them Y2 ECS-80-S-4X

Commit message: Created the board layout
Parts:
- removed U$4: DR73-100-R, Solenoid_parts:DR73-100-R
- added I1: DR73-100-R, Solenoid_parts:DR73-100-R
- moved JP8 122.7 mm to (78.5, 11.9)
- moved JP7 115.8 mm to (78.5, 15.6)
- moved JP6 108.9 mm to (78.5, 19.2)
- moved JP5 102.1 mm to (78.5, 22.9)
- moved R4 90.0 mm to (52.0, 16.3)
- moved U$1 87.3 mm to (58.4, 17.9)
- moved C1 84.8 mm to (45.2, 16.8), turned to 90 degrees
- moved C3 81.3 mm to (56.7, 21.9)
- moved R3 77.2 mm to (42.3, 12.8), turned to 90 degrees
- moved U$2 75.3 mm to (38.0, 13.1)
- moved R2 65.2 mm to (33.4, 11.2)
- moved C21 64.1 mm to (64.9, 45.2), flipped to the top
- moved JP3 63.7 mm to (20.3, 15.6)
- moved CF 62.9 mm to (28.8, 11.2), turned to 180 degrees
- moved R8 61.1 mm to (64.9, 59.9), turned to 270 degrees
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Connections:
- net +5V renamed +3.3V
- net N$1 renamed DRAIN0
- net N$11 renamed FB
- net N$2 renamed DRAIN1
- net N$3 renamed DRAIN2
- net N$4 renamed DRAIN3
- net N$5 renamed DRAIN4
- net N$6 renamed DRAIN5
- net N$7 renamed DRAIN6
- net N$8 renamed DRAIN7
- net N$9 renamed CLR
- removed net N$10: C1.1, R3.2, U$2.5, U$4.1
- removed net N$12: U$2.1, U$3.1, U$4.2
- new net SHDN: R3.1, U$2.4
- new net SW: I1.2, U$2.1, U$3.1
- net +12V: now also C1.1, I1.1, R3.2, U$2.5; no longer R3.1, U$2.4
- net G: now also U$1.G
- net GND: now also C2.2
- net RCK: now also U$1.RCK
- net SER_IN: now also U$1.SER_IN
- net SRCK: now also U$1.SRCK
Routing:
- net +3V3: track 15.3 -> 0.00 mm, vias 3 -> 0
- net NRST: track 14.7 -> 0.00 mm, vias 2 -> 0
- net N$15: track 5.53 -> 0.00 mm
- net OSC_OUT: track 5.15 -> 0.00 mm
- net OSC_IN: track 5.14 -> 0.00 mm
- net N$16: track 3.76 -> 0.00 mm
Other:
- board size 76.2 x 31.8 mm -> 100 x 80 mm

Commit message: Routed most of the board
Parts:
- moved RESET1 66.0 mm to (79.6, 34.2), turned to 90 degrees
- moved C13 57.2 mm to (65.7, 25.4), turned to 270 degrees
- moved R9 55.2 mm to (76.3, 36.1)
- moved C19 54.7 mm to (76.3, 32.7), turned to 270 degrees
- moved C15 54.4 mm to (64.1, 25.4), turned to 270 degrees
- moved C14 37.5 mm to (51.8, 32.8), turned to 180 degrees
- moved R10 35.5 mm to (66.1, 29.3)
- moved C16 35.1 mm to (51.8, 34.4), turned to 180 degrees
- moved C17 31.3 mm to (51.9, 36.2), turned to 180 degrees
- moved C20 30.6 mm to (74.7, 29.3)
- moved C18 28.9 mm to (51.9, 37.8), turned to 180 degrees
- moved R8 27.1 mm to (66.1, 32.8)
- moved Y2 24.2 mm to (70.3, 31.9), turned to 90 degrees
- moved C21 14.5 mm to (74.7, 34.5)
- moved U$8 8.25 mm to (63.7, 35.0), turned to 180 degrees
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Routing:
- net +24V: track 0.00 -> 83.7 mm, vias 0 -> 2
- net DRAIN0: track 0.00 -> 63.8 mm, vias 0 -> 2
- net DRAIN1: track 0.00 -> 59.0 mm, vias 0 -> 2
- net DRAIN2: track 0.00 -> 52.7 mm, vias 0 -> 2
- net GND: track 0.00 -> 47.2 mm, vias 0 -> 2
- net DRAIN3: track 0.00 -> 45.7 mm
- net +3V3: track 0.00 -> 24.8 mm
- net NRST: track 0.00 -> 21.3 mm
- net DRAIN7: track 0.00 -> 18.0 mm
- net SRCK: track 0.00 -> 17.7 mm
- net DRAIN4: track 0.00 -> 17.6 mm
- net DRAIN6: track 0.00 -> 16.7 mm
- net RCK: track 0.00 -> 16.5 mm, vias 0 -> 2
- net SER_IN: track 0.00 -> 16.5 mm
- net DRAIN5: track 0.00 -> 16.3 mm
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
Commit message: Well it's trash but board layout v1 is done
Routing:
- net GND: track 47.2 -> 128.4 mm, vias 2 -> 11
- net NRST: track 21.3 -> 58.7 mm, vias 0 -> 2
- net +3V3: track 24.8 -> 59.9 mm, vias 0 -> 2
- net G: track 0.00 -> 29.7 mm, vias 0 -> 4
- net SWCLK: track 0.00 -> 27.8 mm, vias 0 -> 2
- net SWDIO: track 0.00 -> 24.9 mm, vias 0 -> 2
- net +24V: track 83.7 -> 98.4 mm, vias 2 -> 4
- net +3.3V: track 1.78 -> 16.4 mm, vias 0 -> 4
